Commit message: Update robot_core.xacro

File: description/robot_core.xacro (robot description, xacro)
@@ -1,6 +1,135 @@
 <?xml version="1.0"?>
 <robot xmlns:xacro="http://www.ros.org/wiki/xacro" >
-  <material name="white">
-    <color rgba'"1 1 1 1" />
-  </material>
+    <xacro:include filename="inertial_macros.xacro"/>
+    <material name="white">
+        <color rgba="1 1 1 1" />
+    </material>
+    <material name="orange">
+        <color rgba="1 0.3 0.1 1" />
+    </material>
+    <material name="blue">
+        <color rgba="0.2 0.2 1 1" />
+    </material>
+    <material name="black">
+        <color rgba="0 0 0 1" />
+    </material>
+    <!-- BASE LINK-->
+    <link name="base_link">
+    </link>
+    <!-- CHASSIS LINK-->
+    <joint name="chassis_joint" type="fixed">
+        <parent link="base link"/>
+        <child link="chassis"/>
+        <origin xyz="0 0 0"/>
+    </joint>
+    <link name="chassis">
+        <visual>
+            <origin xyz = "0.15 0 0"/>
+            <geometry>
+                <box size = "0.3 0.3 0.15"/>
+            </geometry>
+            <material name="white"/>
+        </visual>
+        <collision>
+            <origin xyz = "0.15 0 0"/>
+            <geometry>
+                <box size = "0.3 0.3 0.15"/>
+            </geometry>
+        </collision>
+        <xacro:inertial_box mass="0.5" x="0.3" y="0.3" z="0.15">
+            <origin xyz="0.15 0 0" rpy="0 0 0"/>
+        </xacro:inertial_box>
+    </link>
+    <!-- LEFT WHEEL LINK-->
+    <joint name="left_wheel_joint" type="continuous">
+        <parent link="base link"/>
+        <child link="left_wheel"/>
+        <origin xyz="-0.3 0.15 0" rpy="-${pi/2} 0 0"/>
+        <axis xyz="0 0 1"/>
+    </joint>
+    <link name="left_wheel">
+        <visual>
+            <geometry>
+                <cylinder radius="0.05" length="0.04"/>
+            </geometry>
+            <material name="blue"/>
+        </visual>
+        <collision>
+            <geometry>
+                <cylinder radius="0.05" length="0.04"/>
+            </geometry>
+        </collision>
+        <xacro:inertial_cylinder mass="0.1" length="0.04" radius="0.05">
+            <origin xyz="0 0 0" rpy="0 0 0"/>
+        </xacro:inertial_cylinder>
+    </link>
+    <!-- RIGHT WHEEL LINK-->
+    <joint name="right_wheel_joint" type="continuous">
+        <parent link="base link"/>
+        <child link="right_wheel"/>
+        <origin xyz="-0.3 -0.15 0" rpy="${pi/2} 0 0"/>
+        <axis xyz="0 0 -1"/>
+    </joint>
+    <link name="right_wheel">
+        <visual>
+            <geometry>
+                <cylinder radius="0.05" length="0.04"/>
+            </geometry>
+            <material name="blue"/>
+        </visual>
+        <collision>
+            <geometry>
+                <cylinder radius="0.05" length="0.04"/>
+            </geometry>
+        </collision>
+        <xacro:inertial_cylinder mass="0.1" length="0.04" radius="0.05">
+            <origin xyz="0 0 0" rpy="0 0 0"/>
+        </xacro:inertial_cylinder>
+    </link>
+    <!-- LEFT FORWARD WHEEL LINK-->
+    <joint name="left_forward_wheel_joint" type="continuous">
+        <parent link="base link"/>
+        <child link="left_forward_wheel"/>
+        <origin xyz="0 0.15 0" rpy="-${pi/2} 0 0"/>
+        <axis xyz="0 0 1"/>
+    </joint>
+    <link name="left_forward_wheel">
+        <visual>
+            <geometry>
+                <cylinder radius="0.05" length="0.04"/>
+            </geometry>
+            <material name="blue"/>
+        </visual>
+        <collision>
+            <geometry>
+                <cylinder radius="0.05" length="0.04"/>
+            </geometry>
+        </collision>
+        <xacro:inertial_cylinder mass="0.1" length="0.04" radius="0.05">
+            <origin xyz="0 0 0" rpy="0 0 0"/>
+        </xacro:inertial_cylinder>
+    </link>
+    <!-- RIGHT FORWARD WHEEL LINK-->
+    <joint name="right_forward_wheel_joint" type="continuous">
+        <parent link="base link"/>
+        <child link="right_forward_wheel"/>
+        <origin xyz="0 -0.15 0" rpy="${pi/2} 0 0"/>
+        <axis xyz="0 0 -1"/>
+    </joint>
+    <link name="right_forward_wheel">
+        <visual>
+            <geometry>
+                <cylinder radius="0.05" length="0.04"/>
+            </geometry>
+            <material name="blue"/>
+        </visual>
+         <collision>
+            <geometry>
+                <cylinder radius="0.05" length="0.04"/>
+            </geometry>
+        </collision>
+        <xacro:inertial_cylinder mass="0.1" length="0.04" radius="0.05">
+            <origin xyz="0 0 0" rpy="0 0 0"/>
+        </xacro:inertial_cylinder>
+    </link>
 </robot>

Commit message: Update robot_core.xacro

File: description/robot_core.xacro (robot description, xacro)
@@ -41,4 +41,7 @@
         </xacro:inertial_box>
     </link>
+    <gazebo reference ="chassis">
+        <material>Gazebo/White<material/>
+    </gazebo>
     <!-- LEFT WHEEL LINK-->
     <joint name="left_wheel_joint" type="continuous">
@@ -64,4 +67,7 @@
         </xacro:inertial_cylinder>
     </link>
+    <gazebo reference ="left_wheel">
+        <material>Gazebo/Blue<material/>
+    </gazebo>
     <!-- RIGHT WHEEL LINK-->
     <joint name="right_wheel_joint" type="continuous">
@@ -87,4 +93,7 @@
         </xacro:inertial_cylinder>
     </link>
+    <gazebo reference ="right_wheel">
+        <material>Gazebo/Blue<material/>
+    </gazebo>
     <!-- LEFT FORWARD WHEEL LINK-->
     <joint name="left_forward_wheel_joint" type="continuous">
@@ -110,4 +119,7 @@
         </xacro:inertial_cylinder>
     </link>
+    <gazebo reference ="left_forward_wheel">
+        <material>Gazebo/Blue<material/>
+    </gazebo>
     <!-- RIGHT FORWARD WHEEL LINK-->
     <joint name="right_forward_wheel_joint" type="continuous">
@@ -133,3 +145,6 @@
         </xacro:inertial_cylinder>
     </link>
+    <gazebo reference ="right_forward_wheel">
+        <material>Gazebo/Blue<material/>
+    </gazebo>
 </robot>
